File: Design/eInk-picture-frame/eInk-picture-frame.kicad_pcb (KiCad board)
At the start: 2 copper layers, 137 x 115 mm, 13 parts, among them Q1 2N2222, U1 ESP-12E, U2 Push_button, U3 Push_button, U4 Push_button, U5 eInkDisplay_4.3in

Commit message: version 1 complete
Parts:
- added C1: C, Capacitor_THT:C_Disc_D3.0mm_W1.6mm_P2.50mm, B.Cu at (119.4, 121.9)
- added C2: C, Capacitor_THT:C_Disc_D3.0mm_W1.6mm_P2.50mm, B.Cu at (119.4, 127.0)
- added J1: SERIAL, Connector_PinHeader_2.54mm:PinHeader_1x05_P2.54mm_Vertical, B.Cu at (121.9, 49.5)
- added J2: 328_SPI, Connector_PinHeader_2.54mm:PinHeader_1x06_P2.54mm_Vertical, B.Cu at (104.1, 49.5)
- added J3: Conn_01x03_Male, Connector_PinHeader_2.54mm:PinHeader_1x03_P2.54mm_Vertical, B.Cu at (152.4, 49.5)
- added R10: R1, Resistor_THT:R_Axial_DIN0207_L6.3mm_D2.5mm_P10.16mm_Horizontal, B.Cu at (132.1, 68.6)
- added R11: R2, Resistor_THT:R_Axial_DIN0207_L6.3mm_D2.5mm_P10.16mm_Horizontal, B.Cu at (128.3, 78.7)
- added R4: 10k, Resistor_THT:R_Axial_DIN0207_L6.3mm_D2.5mm_P10.16mm_Horizontal, B.Cu at (139.7, 68.6)
- added R5: 10k, Resistor_THT:R_Axial_DIN0207_L6.3mm_D2.5mm_P10.16mm_Horizontal, B.Cu at (135.9, 68.6)
- added R6: 10k, Resistor_THT:R_Axial_DIN0207_L6.3mm_D2.5mm_P10.16mm_Horizontal, B.Cu at (166.4, 78.7)
- added R7: 10k, Resistor_THT:R_Axial_DIN0207_L6.3mm_D2.5mm_P10.16mm_Horizontal, B.Cu at (124.5, 68.6)
- added R8: 100, Resistor_THT:R_Axial_DIN0207_L6.3mm_D2.5mm_P10.16mm_Horizontal, B.Cu at (120.7, 68.6)
- added R9: 10k, Resistor_THT:R_Axial_DIN0207_L6.3mm_D2.5mm_P10.16mm_Horizontal, B.Cu at (179.1, 78.7)
- added U6: 328_RST, kwkong_footprints:6mm_momentary_switch_DIP, B.Cu at (179.1, 49.5)
- added Y1: Crystal, Crystal:Crystal_HC18-U_Vertical, B.Cu at (114.3, 121.9)
- Q1, R1, R2, R3: moved to B.Cu
- U2: value Push_button -> EN; moved to B.Cu
- U3: value Push_button -> BOOT; moved to B.Cu
- U4: value Push_button -> eInkDisplay_4.3in; footprint kwkong_footprints:6mm_momentary_switch_DIP -> Connector_PinHeader_2.54mm:PinHeader_1x06_P2.54mm_Vertical; moved to B.Cu
- U5: value eInkDisplay_4.3in -> ATmega328P-PU; footprint Connector_PinHeader_2.54mm:PinHeader_1x06_P2.54mm_Vertical -> Package_DIP:DIP-28_W7.62mm; moved to B.Cu
- moved R2 300.9 mm to (191.8, 78.7), turned to 90 degrees
- moved R1 266.0 mm to (143.5, 78.7), turned to 90 degrees
- moved U3 256.5 mm to (191.8, 49.5)
- moved U2 218.6 mm to (174.0, 44.5), turned to 180 degrees
- moved U4 176.0 mm to (142.2, 49.5), turned to 90 degrees
- moved U5 175.7 mm to (106.7, 102.9), turned to 180 degrees
- moved Q1 156.7 mm to (111.8, 59.7)
- moved R3 146.3 mm to (90.2, 87.6), turned to 270 degrees
- moved BT2 60.3 mm to (163.8, 135.9), turned to 90 degrees
- moved U1 48.3 mm to (102.9, 78.7)
- moved BT1 17.7 mm to (184.2, 83.8)
- moved BT3 6.84 mm to (143.5, 83.8)
Connections:
- BT1 pad 1: Net-(BT1-Pad1) -> +5V
- BT1 pad 2: Net-(BT1-Pad2) -> +3V3
- BT2 pad 1: Net-(BT2-Pad1) -> +3V3
- BT3 pad 1: Net-(BT3-Pad1) -> Net-(BT2-Pad2)
- BT3 pad 2: Net-(BT3-Pad2) -> GND
- Q1 pad 3: Net-(Q1-Pad3) -> +5V
- R1 pad 1: Net-(R1-Pad1) -> +3V3
- R2 pad 1: Net-(R2-Pad1) -> +3V3
- R3 pad 2: Net-(R3-Pad2) -> GND
- U1 pad 1: Net-(U1-Pad1) -> ESP_WAKE
- U1 pad 15: Net-(U1-Pad15) -> GND
- U1 pad 16: Net-(U1-Pad16) -> Net-(R3-Pad1)
- U1 pad 18: Net-(U1-Pad18) -> Net-(R2-Pad2)
- U1 pad 21: Net-(U1-Pad21) -> 328_RX
- U1 pad 22: Net-(U1-Pad22) -> 328_TX
- U1 pad 3: Net-(U1-Pad3) -> Net-(R6-Pad2)
- U1 pad 4: Net-(U1-Pad4) -> ESP_WAKE
- U1 pad 7: Net-(U1-Pad7) -> eInk_EN
- U1 pad 8: Net-(U1-Pad8) -> +3V3
- U2 pad 2: Net-(U2-Pad2) -> Net-(R6-Pad2)
- U2 pad 4: Net-(U2-Pad4) -> GND
- U3 pad 1: Net-(U3-Pad1) -> Net-(R2-Pad2)
- U3 pad 3: Net-(U3-Pad3) -> GND
- U4 pad 3: Net-(U4-Pad3) -> eInk_DIN
- U4 pad 4: Net-(U4-Pad4) -> eInk_DOUT
- U5 pad 1: Net-(U5-Pad1) -> 328_RST
- U5 pad 2: Net-(U5-Pad2) -> 328_RX
- U5 pad 3: Net-(U5-Pad3) -> 328_TX
- U5 pad 4: Net-(U5-Pad4) -> eInk_DIN
- U5 pad 5: Net-(U5-Pad5) -> eInk_DOUT
- U5 pad 6: Net-(U5-Pad6) -> eInk_EN
Routing:
- net +5V: track 0.00 -> 312.3 mm, vias 0 -> 1
- net +3V3: track 0.00 -> 244.6 mm, vias 0 -> 3
- net 328_RST: track 0.00 -> 152.4 mm, vias 0 -> 7
- net Net-(R2-Pad2): track 0.00 -> 137.8 mm, vias 0 -> 7
- net 328_SCK: track 0.00 -> 105.5 mm
- net 328_MOSI: track 0.00 -> 100.7 mm, vias 0 -> 4
- net 328_MISO: track 0.00 -> 98.2 mm, vias 0 -> 4
- net Net-(R6-Pad2): track 0.00 -> 88.5 mm, vias 0 -> 5
- net eInk_DIN: track 0.00 -> 87.3 mm, vias 0 -> 8
- net eInk_DOUT: track 0.00 -> 86.2 mm, vias 0 -> 6
- net 328_TX: track 0.00 -> 80.3 mm, vias 0 -> 5
- net 328_RX: track 0.00 -> 73.6 mm, vias 0 -> 3
- net Net-(R10-Pad2): track 0.00 -> 65.4 mm, vias 0 -> 3
- net eInk_EN: track 0.00 -> 56.6 mm, vias 0 -> 3
- net Net-(R4-Pad2): track 0.00 -> 41.7 mm, vias 0 -> 5
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- added copper zone on B.Cu, net GND
Other:
- board size 137 x 115 mm -> 157 x 135 mm
- board text added: "--ENSURE CORRECT-- --BATTERY POLARITY!--"
- board text added: "3V3"
- board text added: "5V"
- board text added: "DIN"
- board text added: "DOUT"
- board text added: "GND"
- board text added: "MISO"
- board text added: "MOSI"
- board text added: "RST"
- board text added: "RX"
- board text added: "SCK"
- board text added: "TX"
- board text added: "VCC"
- board text added: "WAKE"
- board text added: "kwkong"
