File: Design/eInk-picture-frame/eInk-picture-frame.sch (KiCad schematic (older format))
At the start: 5 parts

Commit message: still deciding on esp8266 or atmega328
Parts:
- removed BT? (x2): Battery_Cell, symbol Device:Battery_Cell
- added BT2, BT3: Battery_Cell, Battery:BatteryHolder_Keystone_2460_1xAA, symbol Device:Battery_Cell
- added R1, R2, R3, R? (x5): 10k, Resistor_THT:R_Axial_DIN0207_L6.3mm_D2.5mm_P10.16mm_Horizontal, symbol Device:R
- added R?: 100, Resistor_THT:R_Axial_DIN0207_L6.3mm_D2.5mm_P10.16mm_Horizontal, symbol Device:R
- added U3: BOOT, kwkong_footprints:6mm_momentary_switch_DIP, symbol kwkong_symbols:Push_button
- added U?: eInkDisplay_4.3in, symbol kwkong_symbols:eInkDisplay_4.3in
- added U?: EN, kwkong_footprints:6mm_momentary_switch_DIP, symbol kwkong_symbols:Push_button
- BT1: renamed from BT?; footprint (none) -> Battery:BatteryHolder_Keystone_2460_1xAA
- gave numbers to parts that had none: 2
Connections:
- net +5V: now reaches BT1.1 (+)
- net +3V3: now reaches BT1.2 (-)
- net +3V3: now also U1.8 (VCC), BT2.1 (+), R2.1, R?.1, R?.1, R?.1
- net WAKE: now reaches U1.1 (~RST)
- net WAKE: now also U1.4 (GPIO16), R?.2
- net GND: now reaches U1.15 (GND)
- net GND: now also BT3.2 (-), R3.2, R?.2, U3.3, U?.4
- net at U1.16 (GPIO15): now also R3.1
- net at U1.18 (GPIO0): now also R2.2, U3.1
- net at U1.2 (ADC): now also R?.1, R?.2
- net at U1.3 (EN): now also R?.2, U?.2
- new net: BT2.2 (-), BT3.1 (+)
- new net: R?.1, R?.2
Other:
- moved on the sheet: BT1, Q1

Commit message: version 1 complete
Parts:
- removed R1: 10k, Resistor_THT:R_Axial_DIN0207_L6.3mm_D2.5mm_P10.16mm_Horizontal, symbol Device:R
- added C1, C2: C, Capacitor_THT:C_Disc_D3.0mm_W1.6mm_P2.50mm, symbol Device:C
- added J1: SERIAL, Connector_PinHeader_2.54mm:PinHeader_1x05_P2.54mm_Vertical, symbol Connector:Conn_01x05_Male
- added J2: 328_SPI, Connector_PinHeader_2.54mm:PinHeader_1x06_P2.54mm_Vertical, symbol Connector:Conn_01x06_Male
- added J3: Conn_01x03_Male, Connector_PinHeader_2.54mm:PinHeader_1x03_P2.54mm_Vertical, symbol Connector:Conn_01x03_Male
- added R10: R1, Resistor_THT:R_Axial_DIN0207_L6.3mm_D2.5mm_P10.16mm_Horizontal, symbol Device:R
- added R11: R2, Resistor_THT:R_Axial_DIN0207_L6.3mm_D2.5mm_P10.16mm_Horizontal, symbol Device:R
- added R9: 10k, Resistor_THT:R_Axial_DIN0207_L6.3mm_D2.5mm_P10.16mm_Horizontal, symbol Device:R
- added U5: ATmega328P-PU, Package_DIP:DIP-28_W7.62mm, symbol MCU_Microchip_ATmega:ATmega328P-PU
- added U6: 328_RST, kwkong_footprints:6mm_momentary_switch_DIP, symbol kwkong_symbols:Push_button
- added Y1: Crystal, Crystal:Crystal_HC18-U_Vertical, symbol Device:Crystal
- U4: renamed from U?; footprint (none) -> Connector_PinHeader_2.54mm:PinHeader_1x06_P2.54mm_Vertical
- gave numbers to parts that had none: 7
Connections:
- net +3V3: now also J1.2 (Pin_2), J3.2 (Pin_2)
- net +5V: now also Q1.3 (C), J1.1 (Pin_1), J2.1 (Pin_1), J3.1 (Pin_1), R10.1, R9.1, U5.20 (AVCC), U5.7 (VCC)
- net GND: now also U4.5 (GND), C1.2, C2.2, J1.5 (Pin_5), J2.6 (Pin_6), J3.3 (Pin_3), R11.2, U5.22 (GND), U5.8 (GND), U6.3
- net at Q1.1 (E): now also U4.6 (VCC)
- net at Q1.2 (B): now also R8.1
- net 328_RX: now reaches U1.21 (GPIO3/RXD)
- net 328_RX: now also J1.4 (Pin_4), U5.2 (PD0)
- net 328_TX: now reaches U1.22 (GPIO1/TXD)
- net 328_TX: now also J1.3 (Pin_3), U5.3 (PD1)
- net eInk_EN: now reaches U1.7 (GPIO13)
- net eInk_EN: now also R8.2, U5.6 (PD4)
- net eInk_DIN: now reaches U4.3 (DIN)
- net eInk_DIN: now also U5.4 (PD2)
- net eInk_DOUT: now reaches U4.4 (DOUT)
- net eInk_DOUT: now also U5.5 (PD3)
- net WAKE renamed ESP_WAKE
- new net: C2.1, U5.10 (XTAL2/PB7), Y1.2
- new net: R10.2, R11.1, U5.23 (PC0)
- new net: C1.1, U5.9 (XTAL1/PB6), Y1.1
- new net: R9.2, U6.2
- new net 328_MISO: J2.4 (Pin_4), U5.18 (PB4)
- new net 328_MOSI: J2.3 (Pin_3), U5.17 (PB3)
- new net 328_RST: J2.2 (Pin_2), U5.1 (~RESET~/PC6), U6.1
- new net 328_SCK: J2.5 (Pin_5), U5.19 (PB5)
Other:
- moved on the sheet: Q1, R3, R8, U4
